File: SmokeMachine.kicad_pcb (KiCad board)
At the start: 2 copper layers, 14 parts, among them J1 Barrel_Jack, J2 Conn_01x02, J3 Conn_01x02, J4 Conn_01x04, Q1 G30N02T, Q2 G30N02T, U1 LM393, U2 74AUC2G08, U3 74AHCT1G14

Commit message: PCB layout
Parts:
- added C1: 0.1u, Capacitor_SMD:C_0805_2012Metric, F.Cu at (54.0, 60.8)
- added C2: 0.1u, Capacitor_SMD:C_0805_2012Metric, F.Cu at (56.7, 58.8)
- J1: footprint Connector_BarrelJack:BarrelJack_Horizontal -> footprint:mega-fit-1x2
- J2, J3: footprint TerminalBlock:TerminalBlock_bornier-2_P5.08mm -> footprint:mega-fit-1x2
- R1: value R -> 1.1k
- R2, R3: value R -> 1k
- RV1: value R_Potentiometer -> 1k
- TH1: value Thermistor -> 1k->2.2k
- U2: value 74AUC2G08 -> 74HCT2G08DP,125
- U3: value 74AHCT1G14 -> 74AHCT1G14SE-7
- moved J1 42.9 mm to (94.4, 45.8), turned to -90 degrees
- moved RV1 25.7 mm to (57.2, 68.0)
- moved Q1 18.5 mm to (75.5, 55.2), turned to -90 degrees
- moved Q2 17.8 mm to (75.6, 69.5), turned to -90 degrees
- moved TH1 17.8 mm to (45.0, 59.0), turned to -90 degrees
- moved R2 15.5 mm to (56.8, 55.0), turned to -90 degrees
- moved U3 14.7 mm to (63.2, 66.0), turned to 0 degrees
- moved U1 12.4 mm to (62.7, 58.8)
- moved U2 11.8 mm to (69.2, 66.2)
- moved R3 11.2 mm to (54.0, 56.9)
- moved J3 10.4 mm to (94.4, 80.2), turned to -90 degrees
- moved R1 8.31 mm to (56.8, 63.0), turned to -90 degrees
- moved J2 7.92 mm to (94.4, 63.2), turned to -90 degrees
- moved J4 5.30 mm to (45.2, 70.0)
Connections:
- J1 pad 2: GND -> GND1
- J2 pad 2: GND -> GND1
- J3 pad 2: GND -> GND1
- RV1 pad 1: GND -> Net-(R1-Pad2)
- RV1 pad 2: unconnected-(RV1-Pad2) -> GND
- RV1 pad 3: Net-(R1-Pad2) -> GND
Routing:
- net 12V: track 0.00 -> 45.6 mm
- net GND1: track 0.00 -> 44.7 mm
- net ME: track 0.00 -> 29.7 mm, vias 0 -> 2
- net EE: track 0.00 -> 25.9 mm
- net Net-(U1-Pad1): track 0.00 -> 19.7 mm
- net Net-(U1A-+): track 0.00 -> 17.9 mm
- net Net-(J3-Pin_1): track 0.00 -> 15.5 mm
- net Net-(J2-Pin_1): track 0.00 -> 14.4 mm
- net Net-(Q1-G): track 0.00 -> 14.4 mm
- net GND: track 0.00 -> 10.9 mm, vias 0 -> 5
- net Net-(U2-Pad5): track 0.00 -> 8.11 mm
- net Net-(Q2-G): track 0.00 -> 7.91 mm
- net Net-(R1-Pad2): track 0.00 -> 4.29 mm
- net Net-(U1A--): track 0.00 -> 3.66 mm
- added copper zone on F.Cu, net 5V

Commit message: Flyback diode
Parts:
- added D1: 1N4004, Diode_THT:D_DO-41_SOD81_P10.16mm_Horizontal, F.Cu at (71.9, 85.5)
- added G***: LOGO, footprint:logo, F.Cu at (63.0, 42.0)
- added REF**: mounting_hole_3mm, footprint:mounting_hole_3mm, F.Cu at (104.0, 87.0)
- added REF**: mounting_hole_3mm, footprint:mounting_hole_3mm, F.Cu at (38.0, 87.0)
- added REF**: mounting_hole_3mm, footprint:mounting_hole_3mm, F.Cu at (38.0, 38.0)
- added REF**: mounting_hole_3mm, footprint:mounting_hole_3mm, F.Cu at (104.0, 38.0)
- J4: value Conn_01x04 -> Conn_01x06; footprint footprint:mini-lock-4x1 -> footprint:mini-lock-6x1-vert
- moved J4 2.76 mm to (45.0, 72.8)
Connections:
- C1 pad 1: Net-(U1A-+) -> REF
- C2 pad 1: Net-(U1A-+) -> REF
- J1 pad 2: GND1 -> GND
- J2 pad 2: GND1 -> GND
- J3 pad 2: GND1 -> GND
- J4 pad 4: GND -> REF
- R1 pad 1: Net-(U1A-+) -> REF
- TH1 pad 2: Net-(U1A-+) -> REF
- U1 pad 3: Net-(U1A-+) -> REF
Routing:
- net GND: track 10.9 -> 70.9 mm
- net GND1: track 44.7 -> 0.00 mm
- net REF: track 0.00 -> 30.1 mm
- net Net-(U1A-+): track 17.9 -> 0.00 mm
- net Net-(D1-K): track 15.5 -> 28.0 mm
- net Net-(U1A--): track 3.66 -> 8.40 mm
- net EE: track 25.9 -> 27.7 mm
- net 5V: track 0.00 -> 1.82 mm
- net Net-(Q1-G): track 14.4 -> 13.8 mm
- net ME: track 29.7 -> 30.2 mm
Other:
- board outline added: 72 x 55 mm
- board text added: "Smoke Machine Controller v1.0"

Commit message: PCB update
Parts:
- TH1: footprint footprint:mini-lock-2x1 -> footprint:mini-lock-2x1-vert
- moved D1 10.6 mm to (81.6, 81.1), turned to 180 degrees
- moved Q1 6.01 mm to (79.2, 59.9), turned to 90 degrees
- moved Q2 5.68 mm to (79.1, 73.9), turned to 90 degrees
- turned J4 to -90 degrees
Connections:
- D1 pad 1: Net-(D1-K) -> 12V
- D1 pad 2: GND -> Net-(D1-A)
- J1 pad 1: 12V -> GND
- J1 pad 2: GND -> 12V
- J2 pad 2: GND -> 12V
- J3 pad 1: Net-(D1-K) -> Net-(D1-A)
- J3 pad 2: GND -> 12V
- Q1 pad 2: 12V -> Net-(J2-Pin_1)
- Q1 pad 3: Net-(J2-Pin_1) -> GND
- Q2 pad 2: 12V -> Net-(D1-A)
- Q2 pad 3: Net-(D1-K) -> GND
- TH1 pad 1: 5V -> REF
- TH1 pad 2: REF -> 5V
Routing:
- net Net-(D1-A): track 0.00 -> 33.0 mm
- net Net-(D1-K): track 28.0 -> 0.00 mm
- net GND: track 70.9 -> 50.3 mm
- net 12V: track 45.6 -> 65.6 mm
- net Net-(Q2-G): track 7.91 -> 12.6 mm
- net Net-(J2-Pin_1): track 14.4 -> 11.9 mm
- net 5V: track 1.82 -> 0.00 mm
- net Net-(Q1-G): track 13.8 -> 12.4 mm
- net ME: vias 2 -> 4
- net EE: vias 0 -> 2
Other:
- board text added: "+ -"
- board text added: "- NC REF ME EE +"
- board text added: "Rth"
- board text added: "element"
- board text added: "input"
- board text added: "pump"
