File: SmokeMachine.kicad_sch (KiCad schematic)
At the start: 6 parts, among them U1 LM393

Commit message: Add files via upload
Parts:
- removed RV1: 1k, symbol Device:R_Potentiometer_Trim
- added J1: Barrel_Jack, Connector_BarrelJack:BarrelJack_Horizontal, symbol Connector:Barrel_Jack
- added J2, J3: Conn_01x02, TerminalBlock:TerminalBlock_bornier-2_P5.08mm, symbol Connector_Generic:Conn_01x02
- added J4: Conn_01x04, footprint:mini-lock-4x1, symbol Connector_Generic:Conn_01x04
- added Q1, Q2: G30N02T, Package_TO_SOT_THT:TO-220-3_Vertical, symbol Device:Q_NMOS_GDS
- added RV1: R_Potentiometer, Potentiometer_THT:Potentiometer_Bourns_3296W_Vertical, symbol Device:R_Potentiometer
- added U2: 74AUC2G08, symbol 74xGxx:74AUC2G08
- added U3: 74AHCT1G14, Package_TO_SOT_SMD:SOT-353_SC-70-5, symbol 74xGxx:74LVC1GU04DRL
- R1: value 1.15k -> R; footprint (none) -> Resistor_SMD:R_0805_2012Metric
- R2, R3: value 1k -> R; footprint (none) -> Resistor_SMD:R_0805_2012Metric
- TH1: value 1k -> Thermistor; footprint (none) -> footprint:mini-lock-2x1
- U1: footprint (none) -> Package_SO:SOIC-8_3.9x4.9mm_P1.27mm
Connections:
- net GND: now also J1.2, J2.2 (Pin_2), J3.2 (Pin_2), J4.4 (Pin_4), RV1.1, U2.4 (GND), U3.3 (GND)
- net at TH1.2, U1.3 (+): now also R1.1; no longer R1.2
- net at U1.1: now also U2.1, U3.2
- net +5V renamed 5V
- net 5V: now also J4.1 (Pin_1), U2.8 (VCC), U3.5 (VCC)
- new net: Q2.1 (G), U2.3
- new net: U2.5, U3.4
- new net: R1.2, RV1.3
- new net: J2.1 (Pin_1), Q1.3 (S)
- new net: Q1.1 (G), U2.7
- new net: J3.1 (Pin_1), Q2.3 (S)
- new net 12V: J1.1, Q1.2 (D), Q2.2 (D)
- new net EE: J4.2 (Pin_2), U2.2
- new net ME: J4.3 (Pin_3), U2.6
Other:
- note removed: "R1 -> current limiting, when Rpot = 0 Rv1 -> adjust temperature set-point"
- note removed: "TH1 R@0 = 1k R@300 = 2.12k"

Commit message: PCB layout
Parts:
- added C1, C2: 0.1u, Capacitor_SMD:C_0805_2012Metric, symbol Device:C_Small
- J1: footprint Connector_BarrelJack:BarrelJack_Horizontal -> footprint:mega-fit-1x2
- J2, J3: footprint TerminalBlock:TerminalBlock_bornier-2_P5.08mm -> footprint:mega-fit-1x2
- R1: value R -> 1.1k
- R2, R3: value R -> 1k
- RV1: value R_Potentiometer -> 1k
- TH1: value Thermistor -> 1k->2.2k
- U2: value 74AUC2G08 -> 74HCT2G08DP,125; footprint (none) -> Package_SO:TSSOP-8_3x3mm_P0.65mm
- U2: value 74AUC2G08 -> 74HCT2G08DP,125
- U3: value 74AHCT1G14 -> 74AHCT1G14SE-7
Connections:
- net GND: now also RV1.2, RV1.3, C1.2; no longer J1.2, J2.2 (Pin_2), J3.2 (Pin_2), RV1.1
- net at R1.1, TH1.2, U1.3 (+): now also C1.1, C2.1
- net at R1.2: now also RV1.1; no longer RV1.3
- net at R2.2, R3.1, U1.2 (-): now also C2.2
- new net GND1: J1.2, J2.2 (Pin_2), J3.2 (Pin_2)
Other:
- note added: "Heating element connector, up to 10A current"
- note added: "Pump motor connector, <1A current"
- moved on the sheet: J1, J2, J3, J4, Q1, Q2, R1, R2, R3, RV1, TH1, U1A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

Commit message: Flyback diode
Parts:
- removed J4: Conn_01x04, footprint:mini-lock-4x1, symbol Connector_Generic:Conn_01x04
- added D1: 1N4004, Diode_THT:D_DO-41_SOD81_P10.16mm_Horizontal, symbol Diode:1N4004
- added J4: Conn_01x06, footprint:mini-lock-6x1-vert, symbol Connector_Generic:Conn_01x06
Connections:
- net GND1 is gone; now on net GND: J1.2, J2.2 (Pin_2), J3.2 (Pin_2)
- net 5V: now also J4.1 (Pin_1)
- net EE: now also J4.2 (Pin_2)
- net GND: now also D1.2 (A), J4.6 (Pin_6)
- net ME: now also J4.3 (Pin_3)
- net REF: now reaches C1.1, C2.1, R1.1, TH1.2, U1.3 (+)
- net REF: now also J4.4 (Pin_4)
- net at J3.1 (Pin_1), Q2.3 (S): now also D1.1 (K)
Other:
- moved on the sheet: U2C

Commit message: PCB update
Parts:
- TH1: footprint footprint:mini-lock-2x1 -> footprint:mini-lock-2x1-vert
Connections:
- net 12V: now also D1.1 (K), J1.2, J2.2 (Pin_2), J3.2 (Pin_2); no longer J1.1, Q1.2 (D), Q2.2 (D)
- net 5V: now also TH1.2; no longer TH1.1
- net GND: now also J1.1, Q1.3 (S), Q2.3 (S); no longer D1.2 (A), J1.2, J2.2 (Pin_2), J3.2 (Pin_2)
- net REF: now also TH1.1; no longer TH1.2
- net at J2.1 (Pin_1): now also Q1.2 (D); no longer Q1.3 (S)
- new net: D1.2 (A), J3.1 (Pin_1), Q2.2 (D)
